Commit message: Cambio de nombre

File: src/suv_modelo/urdf/suv.xacro (robot description, xacro)
@@ -1,4 +1,4 @@
 <?xml version="1.0"?>
-<robot name="Camion" xmlns:xacro="http://www.ros.org/wiki/xacro" >
+<robot name="Suv" xmlns:xacro="http://www.ros.org/wiki/xacro" >
 	<xacro:property name="camera_link" value="0.05" /> <!-- Size of square 'camera' box -->
 	<xacro:property name="pi" value="3.1415" />
@@ -9,5 +9,5 @@
 		<origin xyz="${0.093*reflect} -0.13993 0" rpy="1.5708 1.5708 0" />
 	</xacro:macro>
-	<xacro:macro name="CamionPos" >
+	<xacro:macro name="SuvPos" >
 		<origin xyz="0 0 0" rpy="${pi/2} 0 0" />
 	</xacro:macro>
@@ -16,8 +16,8 @@
 	</xacro:macro>
    <!-- Import all Gazebo-customization elements, including Gazebo colors -->
-   <xacro:include filename="$(find camion_modelo)/urdf/camion.gazebo" />
-   <xacro:include filename="$(find camion_modelo)/urdf/camion.transmission" />
+   <xacro:include filename="$(find suv_modelo)/urdf/suv.gazebo" />
+   <xacro:include filename="$(find suv_modelo)/urdf/suv.transmission" />
 	<link
-    name="Camion">
+    name="Suv">
     <inertial>
       <origin
@@ -35,8 +35,8 @@
     </inertial>
     <visual>
-      <xacro:CamionPos />
-      <geometry>
-        <mesh
-          filename="package://camion_modelo/meshes/Camion.stl" />
+      <xacro:SuvPos />
+      <geometry>
+        <mesh
+          filename="package://suv_modelo/meshes/suv.stl" />
       </geometry>
       <material
@@ -47,8 +47,8 @@
     </visual>
     <collision>
-      <xacro:CamionPos />
-      <geometry>
-        <mesh
-          filename="package://camion_modelo/meshes/Camion.stl" />
+      <xacro:SuvPos />
+      <geometry>
+        <mesh
+          filename="package://suv_modelo/meshes/suv.stl" />
       </geometry>
     </collision>
@@ -74,17 +74,17 @@
       <geometry>
         <mesh
-          filename="package://camion_modelo/meshes/FrontL.stl" />
-      </geometry>
-      <material
-        name="">
-        <color
-          rgba="0.0078431 0 0.019608 1" />
-      </material>
-    </visual>
-    <collision>
-      <xacro:WheelPos reflect="0" />
-      <geometry>
-        <mesh
-          filename="package://camion_modelo/meshes/FrontL.stl" />
+          filename="package://suv_modelo/meshes/FrontL.stl" />
+      </geometry>
+      <material
+        name="">
+        <color
+          rgba="0.0078431 0 0.019608 1" />
+      </material>
+    </visual>
+    <collision>
+      <xacro:WheelPos reflect="0" />
+      <geometry>
+        <mesh
+          filename="package://suv_modelo/meshes/FrontL.stl" />
       </geometry>
     </collision>
@@ -95,5 +95,5 @@
     <xacro:RwheelOrigin reflect="1" />
     <parent
-      link="Camion" />
+      link="Suv" />
     <child
       link="FrontL" />
@@ -121,17 +121,17 @@
       <geometry>
         <mesh
-          filename="package://camion_modelo/meshes/FrontR.stl" />
-      </geometry>
-      <material
-        name="">
-        <color
-          rgba="0.0078431 0 0.019608 1" />
-      </material>
-    </visual>
-    <collision>
-      <xacro:WheelPos reflect="1" />
-      <geometry>
-        <mesh
-          filename="package://camion_modelo/meshes/FrontR.stl" />
+          filename="package://suv_modelo/meshes/FrontR.stl" />
+      </geometry>
+      <material
+        name="">
+        <color
+          rgba="0.0078431 0 0.019608 1" />
+      </material>
+    </visual>
+    <collision>
+      <xacro:WheelPos reflect="1" />
+      <geometry>
+        <mesh
+          filename="package://suv_modelo/meshes/FrontR.stl" />
       </geometry>
     </collision>
@@ -142,5 +142,5 @@
     <xacro:RwheelOrigin reflect="-1" />
     <parent
-      link="Camion" />
+      link="Suv" />
     <child
       link="FrontR" />
@@ -168,17 +168,17 @@
       <geometry>
         <mesh
-          filename="package://camion_modelo/meshes/RearL.stl" />
-      </geometry>
-      <material
-        name="">
-        <color
-          rgba="0.0078431 0 0.019608 1" />
-      </material>
-    </visual>
-    <collision>
-      <xacro:WheelPos reflect="0" />
-      <geometry>
-        <mesh
-          filename="package://camion_modelo/meshes/RearL.stl" />
+          filename="package://suv_modelo/meshes/RearL.stl" />
+      </geometry>
+      <material
+        name="">
+        <color
+          rgba="0.0078431 0 0.019608 1" />
+      </material>
+    </visual>
+    <collision>
+      <xacro:WheelPos reflect="0" />
+      <geometry>
+        <mesh
+          filename="package://suv_modelo/meshes/RearL.stl" />
       </geometry>
     </collision>
@@ -189,5 +189,5 @@
     <xacro:FwheelOrigin reflect="1" />
     <parent
-      link="Camion" />
+      link="Suv" />
     <child
       link="RearL" />
@@ -215,5 +215,5 @@
       <geometry>
         <mesh
-          filename="package://camion_modelo/meshes/RearR.stl" />
+          filename="package://suv_modelo/meshes/RearR.stl" />
       </geometry>
       <material
@@ -227,5 +227,5 @@
       <geometry>
         <mesh
-          filename="package://camion_modelo/meshes/RearR.stl" />
+          filename="package://suv_modelo/meshes/RearR.stl" />
       </geometry>
     </collision>
@@ -236,5 +236,5 @@
     <xacro:FwheelOrigin reflect="-1" />
     <parent
-      link="Camion" />
+      link="Suv" />
     <child
       link="RearR" />
@@ -245,5 +245,5 @@
     <axis xyz="0 1 0" />
     <origin xyz="0 -0.23 0.06" rpy="0 0 ${-1*pi/2}"/>
-    <parent link="Camion"/>
+    <parent link="Suv"/>
     <child link="camera_link"/>
   </joint>
